File: hotglue-beetle-screw-switch.kicad_sch (KiCad schematic)
At the start: 11 parts, among them J1 Conn_01x02_Pin, J2 Conn_01x02_Socket, J3 Conn_01x02_Socket, J4 Conn_01x02_Socket

Commit message: plotted gerbers for intial design. Began fix for incorrect footprint on Wurth standoff. Backup after PC crash and recovery
Parts:
- H2, H3: footprint Mounting_Wuerth:Mounting_Wuerth_WA-SMSI-M3_H3mm_9774030360 -> Trent-footprints:MP_Wurth_WP-SMBU_746600330
